File: pcbs/my_first_keyboard_wireless_autorouted.kicad_pcb (KiCad board)
At the start: 2 copper layers, 135.9 x 108 mm, 78 parts

Commit message: v1
Parts:
- moved D20 0.10 mm to (170.4, 109.8)
- moved D1 0.10 mm to (92.2, 98.5)
- moved D10 0.10 mm to (149.2, 84.2)
- moved D11 0.10 mm to (149.2, 65.2)
- moved D12 0.10 mm to (149.2, 46.2)
- moved D13 0.10 mm to (168.2, 87.4)
- moved D14 0.10 mm to (168.2, 68.4)
- moved D15 0.10 mm to (168.2, 49.4)
- moved D16 0.10 mm to (187.2, 89.8)
- moved D17 0.10 mm to (187.2, 70.8)
- moved D18 0.10 mm to (187.2, 51.8)
- moved D19 0.10 mm to (149.2, 109.2)
- moved D2 0.10 mm to (92.2, 79.5)
- moved D23 0.10 mm to (107.8, 98.5)
- moved D24 0.10 mm to (107.8, 79.5)
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Routing:
- net R3: track 198.2 -> 155.8 mm
- net R1: track 161.8 -> 187.8 mm, vias 7 -> 6
- net R2: track 170.8 -> 196.5 mm, vias 8 -> 5
- net C2: track 210.5 -> 186.8 mm, vias 5 -> 4
- net C3: track 173.4 -> 187.2 mm, vias 4 -> 5
- net C0: track 187.5 -> 197.1 mm
- net GND: track 128.0 -> 137.3 mm, vias 3 -> 2
- net R0: track 203.1 -> 197.0 mm
- net VCC: track 35.5 -> 40.8 mm, vias 0 -> 1
- net C1: track 172.6 -> 167.4 mm, vias 4 -> 3
- net RST: track 41.1 -> 46.2 mm, vias 1 -> 0
- net RAW: track 58.8 -> 63.8 mm, vias 1 -> 3
- net C5: track 146.9 -> 143.2 mm
- net CS: track 51.4 -> 48.7 mm
- net BAT_P: track 18.3 -> 16.3 mm
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